Commit message: feat: fix bug

File: urdf/robot.urdf (robot description, URDF)
Before this commit: robot arpis, 35 links, 34 joints
Joints:
- joint head_pan: axis 0 1 0 -> 0 0 1
- joint left_shoulder_roll: axis 0 0 1 -> 0 1 0; origin xyz=0 .0 -0.15 rpy=0 0 0 -> xyz=0 .0 -0.15 rpy=0 0.3 0
- joint right_shoulder_roll: axis 0 0 1 -> 0 1 0; origin xyz=0 .0 -0.15 rpy=0 0 0 -> xyz=0 .0 -0.15 rpy=0 0.3 0

Commit message: fix: fix urdf

File: urdf/robot.urdf (robot description, URDF)
Before this commit: robot arpis, 35 links, 34 joints
Joints:
- joint left_shoulder_roll: origin xyz=0 .0 -0.15 rpy=0 0.3 0 -> xyz=0 .0 -0.15 rpy=0 0.35 0
- joint right_shoulder_roll: origin xyz=0 .0 -0.15 rpy=0 0.3 0 -> xyz=0 .0 -0.15 rpy=0 -0.35 0
